Commit message: change limits in jLeftShoulder_rotz and jRightShoulder_rotz

File: src/humanmodelgenerator/models/humanModelTemplate/humanModelTemplate.urdf (robot description, URDF)
Before this commit: robot HumanModel, 133 links, 132 joints
Joints:
- joint jLeftShoulder_rotz: limit lower=-3.14159 upper=0.785398 effort=30 velocity=1.0 -> lower=-1.91986 upper=0.785398 effort=30 velocity=1.0
- joint jRightShoulder_rotz: limit lower=-0.785398 upper=3.14159 effort=30 velocity=1.0 -> lower=-0.785398 upper=1.91986 effort=30 velocity=1.0
